File: DMH_Output_PANEL/DMH_Output_PANEL.kicad_pcb (KiCad board)
At the start: 2 copper layers, 50 x 200 mm, 5 parts, among them J0 Panel_GND_Solder_Wire_Pad

Commit message: Panel design in progress
Parts:
- added H10: Ext In R, SynthStuff:Jack_6.35mm_Cutout_v3, F.Cu at (151.8, 115.0)
- added H11: Euro L, SynthStuff:Jack_6.35mm_Cutout_Output_v6, F.Cu at (168.9, 80.8)
- added H12: Euro R, SynthStuff:Jack_6.35mm_Cutout_Output_v6, F.Cu at (168.9, 97.9)
- added H13: Out HP, SynthStuff:Jack_6.35mm_Cutout_Output_v6, F.Cu at (58.5, 208.8)
- added H14: HP Volume, SynthStuff:Pot_Cutout_Tiny, F.Cu at (176.4, 136.3)
- added H15: Volume, SynthStuff:Pot_Cutout_Medium, F.Cu at (144.9, 142.3)
- added H5: In L, SynthStuff:Jack_6.35mm_Cutout_v3, F.Cu at (75.0, 190.2)
- added H6: In R, SynthStuff:Jack_6.35mm_Cutout_v3, F.Cu at (91.5, 190.2)
- added H7: Out L, SynthStuff:Jack_6.35mm_Cutout_Output_v6, F.Cu at (75.0, 208.8)
- added H8: Out R, SynthStuff:Jack_6.35mm_Cutout_Output_v6, F.Cu at (91.5, 208.8)
- added H9: Ext In L, SynthStuff:Jack_6.35mm_Cutout_v3, F.Cu at (151.8, 97.9)
Other:
- board text added: "5532"
- board text added: "Output"
- board text removed: "Module Name"
- board text removed: "TYPE"
