File: DMH_Output_PANEL/DMH_Output_PANEL.kicad_sch (KiCad schematic)
At the start: 5 parts, among them J0 Panel_GND_Solder_Wire_Pad

Commit message: Panel design in progress
Parts:
- added H10: Ext In R, SynthStuff:Jack_6.35mm_Cutout_v3, symbol SynthStuff:MountingHole_Jack6.35mm_v2
- added H11: Euro L, SynthStuff:Jack_6.35mm_Cutout_Output_v6, symbol SynthStuff:MountingHole_Jack6.35mm_Output_v2
- added H12: Euro R, SynthStuff:Jack_6.35mm_Cutout_Output_v6, symbol SynthStuff:MountingHole_Jack6.35mm_Output_v2
- added H13: Out HP, SynthStuff:Jack_6.35mm_Cutout_Output_v6, symbol SynthStuff:MountingHole_Jack6.35mm_Output_v2
- added H14: HP Volume, SynthStuff:Pot_Cutout_Tiny, symbol SynthStuff:MountingHole_Pot
- added H15: Volume, SynthStuff:Pot_Cutout_Medium, symbol SynthStuff:MountingHole_Pot
- added H5: In L, SynthStuff:Jack_6.35mm_Cutout_v3, symbol SynthStuff:MountingHole_Jack6.35mm_v2
- added H6: In R, SynthStuff:Jack_6.35mm_Cutout_v3, symbol SynthStuff:MountingHole_Jack6.35mm_v2
- added H7: Out L, SynthStuff:Jack_6.35mm_Cutout_Output_v6, symbol SynthStuff:MountingHole_Jack6.35mm_Output_v2
- added H8: Out R, SynthStuff:Jack_6.35mm_Cutout_Output_v6, symbol SynthStuff:MountingHole_Jack6.35mm_Output_v2
- added H9: Ext In L, SynthStuff:Jack_6.35mm_Cutout_v3, symbol SynthStuff:MountingHole_Jack6.35mm_v2
Connections:
- net GND: now also H10.1, H11.1, H12.1, H13.1, H14.1, H15.1, H5.1, H6.1, H7.1, H8.1, H9.1
