File: DMH_Output_PCB_1/Output_Meter.kicad_sch (KiCad schematic)
At the start: 63 parts, among them Q1 BC558, Q2 BC558, U1 TL072, U2 LM339, U3 LM339, U4 LM339, U5 LM339, U6 LM339

Commit message: Adjustments during breadboarding
Parts:
- R21, R23: value 180R -> 100R
- R22, R25: value 3k3 -> 470R
Other:
- note added: "Need 470R here, otherwise the first LED on the left will never switch off"
Changed lines of the file:
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@@
 		(comment 1 "PCB for 5 cm Kosmo format synthesizer module")
 	)
+	(circle
+		(center 173.99 162.56)
+		(radius 6.4758)
+		(stroke
+			(width 0)
+			(type default)
+		)
+		(fill
+			(type none)
+		)
+	)
+	(text "Need 470R here, otherwise the first LED\non the left will never switch off"
+		(exclude_from_sim no)
+		(at 200.66 164.338 0)
+		(effects
+			(font
+				(size 1.27 1.27)
+			)
+		)
+	)
 	(junction
 		(at 139.7 139.7)
@@
 			)
 		)
-		(property "Value" "3k3"
+		(property "Value" "470R"
 			(at 247.65 156.21 90)
 			(effects
@@
 			)
 		)
-		(property "Value" "180R"
+		(property "Value" "100R"
 			(at 251.46 128.2699 0)
 			(effects
@@
 			)
 		)
-		(property "Value" "3k3"
+		(property "Value" "470R"
 			(at 95.25 156.21 90)
 			(effects
@@
 			)
 		)
-		(property "Value" "180R"
+		(property "Value" "100R"
 			(at 91.44 128.2699 0)
 			(effects
