File: DMH_Output_PCB_Main/Pregain_stage.kicad_sch (KiCad schematic)
At the start: 9 parts, among them U7 TL072

Commit message: Prep for Main and MZ PCBs design in progress
Connections:
- net L_Monitor renamed L_Monitor_M
- net Left_In renamed L_In_M
- net R_Monitor renamed R_Monitor_M
- net Right In renamed R_In_M
Changed lines of the file:
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@@
 		)
 	)
-	(hierarchical_label "R_Monitor"
+	(hierarchical_label "R_Monitor_M"
 		(shape output)
 		(at 116.84 127 0)
@@
 		)
 	)
-	(hierarchical_label "Left_In"
+	(hierarchical_label "L_In_M"
 		(shape input)
 		(at 60.96 60.96 180)
@@
 		)
 	)
-	(hierarchical_label "Right In"
+	(hierarchical_label "R_In_M"
 		(shape input)
 		(at 60.96 124.46 180)
@@
 		)
 	)
-	(hierarchical_label "L_Monitor"
+	(hierarchical_label "L_Monitor_M"
 		(shape output)
 		(at 116.84 63.5 0)

Commit message: Prepped for Main PCB design
Parts:
- added J29: Conn_01x04_PinHeader, Connector_PinSocket_2.54mm:PinSocket_1x04_P2.54mm_Vertical, symbol SynthStuff:Conn_01x04_PinHeader
- added J30: Conn_01x04_PinHeader, Connector_PinHeader_2.54mm:PinHeader_1x04_P2.54mm_Vertical, symbol SynthStuff:Conn_01x04_PinHeader
Connections:
- net L_In_M: now also J29.1 (Pin_1); no longer R26.1
- net L_Monitor_M: now also J29.3 (Pin_3); no longer C7.2
- net R_In_M: now also J29.2 (Pin_2); no longer R29.1
- net R_Monitor_M: now also J29.4 (Pin_4); no longer C10.2
- new net: C7.2, J30.3 (Pin_3)
- new net: J30.2 (Pin_2), R29.1
- new net: C10.2, J30.4 (Pin_4)
- new net: J30.1 (Pin_1), R26.1
Other:
- note added: "Mezanine PCB"
