File: DMH_Output_PCB_Main/Balanced_line_driver.kicad_sch (KiCad schematic)
At the start: 40 parts, among them J31 Conn_01x06_PinHeader, J32 Conn_01x06_PinHeader, U10 NE5532, U9 NE5532

Commit message: Inverted line outputs hot and cold pins
... in order to avoid phase inversion at the TRS jack tip.
Connections:
- net L_Bal_OUT_N_M: now also J31.3 (Pin_3); no longer J31.4 (Pin_4)
- net L_Bal_OUT_P_M: now also J31.4 (Pin_4); no longer J31.3 (Pin_3)
- net R_Bal_OUT_N_M: now also J31.5 (Pin_5); no longer J31.6 (Pin_6)
- net R_Bal_OUT_P_M: now also J31.6 (Pin_6); no longer J31.5 (Pin_5)
Changed lines of the file:
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@@
 	(hierarchical_label "R_Bal_OUT_N_M"
+		(shape output)
+		(at 177.8 165.1 0)
+		(effects
+			(font
+				(size 1.27 1.27)
+			)
+			(justify left)
+		)
+	)
+	(hierarchical_label "R_Bal_OUT_P_M"
 		(shape output)
 		(at 177.8 215.9 0)
@@
 		)
 	)
-	(hierarchical_label "R_Bal_OUT_P_M"
-		(shape output)
-		(at 177.8 165.1 0)
-		(effects
-			(font
-				(size 1.27 1.27)
-			)
-			(justify left)
-		)
-	)
 	(hierarchical_label "L_Bal_OUT_P_M"
 		(shape output)
-		(at 177.8 50.8 0)
+		(at 177.8 101.6 0)
 		(effects
 			(font
@@
 	(hierarchical_label "L_Bal_OUT_N_M"
 		(shape output)
-		(at 177.8 101.6 0)
+		(at 177.8 50.8 0)
 		(effects
 			(font

Commit message: Exported BoM and Schematic
Other:
- company: (none) -> DMH Instruments
- title: (none) -> 5532 Output
Changed lines of the file:
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@@
 	(paper "A4" portrait)
 	(title_block
-		(comment 1 "PCB for 5 cm Kosmo format synthesizer module")
+		(title "5532 Output")
+		(date "2026-07-09")
+		(company "DMH Instruments")
+		(comment 1 "5 cm Kosmo format synthesizer module")
 	)
 	(rectangle
