File: DMH_Output_PCB_Main/Headphone_amplifier.kicad_sch (KiCad schematic)
At the start: 21 parts, among them J12 Conn_01x06_PinHeader, J27 Conn_01x06_PinHeader, J38 Conn_01x06, U11 TL074, U13 NE5532, U15 NE5532

Commit message: Exported BoM and Schematic
Other:
- company: (none) -> DMH Instruments
- title: (none) -> 5532 Output
Changed lines of the file:
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@@
 	(paper "A4")
 	(title_block
-		(comment 1 "PCB for 5 cm Kosmo format synthesizer module")
+		(title "5532 Output")
+		(date "2026-07-09")
+		(company "DMH Instruments")
+		(comment 1 "5 cm Kosmo format synthesizer module")
 	)
 	(rectangle
