File: DMH_Output_PCB_Main/Input_Meter.kicad_sch (KiCad schematic)
At the start: 29 parts, among them U20 TL072, U24 LM339, U25 LM339

Commit message: Fixed 22k resistor value
Parts:
- R84: value 22K -> 22k
Changed lines of the file:
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@@
 			)
 		)
-		(property "Value" "22K"
+		(property "Value" "22k"
 			(at 57.15 21.59 90)
 			(show_name no)

Commit message: Adjusted output meter resistors
... and deleted unnecessary notes
Other:
- note removed: "Was 100k"
- note removed: "Was 20k"
Changed lines of the file:
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@@
 		(comment 1 "PCB for 5 cm Kosmo format synthesizer module")
-	)
-	(circle
-		(center 171.45 22.86)
-		(radius 5.08)
-		(stroke
-			(width 0)
-			(type default)
-		)
-		(fill
-			(type none)
-		)
-	)
-	(circle
-		(center 57.15 22.86)
-		(radius 5.08)
-		(stroke
-			(width 0)
-			(type default)
-		)
-		(fill
-			(type none)
-		)
-	)
-	(circle
-		(center 146.05 45.72)
-		(radius 5.08)
-		(stroke
-			(width 0)
-			(type default)
-		)
-		(fill
-			(type none)
-		)
 	)
 	(rectangle
@@
 		)
 	)
-	(circle
-		(center 31.75 45.72)
-		(radius 5.08)
-		(stroke
-			(width 0)
-			(type default)
-		)
-		(fill
-			(type none)
-		)
-	)
 	(text "3 = Green"
 		(exclude_from_sim no)
 		(at 91.44 108.458 0)
-		(effects
-			(font
-				(size 1.27 1.27)
-			)
-		)
-	)
-	(text "Was 100k"
-		(exclude_from_sim no)
-		(at 57.15 16.51 0)
-		(effects
-			(font
-				(size 1.27 1.27)
-			)
-		)
-	)
-	(text "Was 20k"
-		(exclude_from_sim no)
-		(at 31.75 39.37 0)
 		(effects
 			(font
@@
 		(effects
 			(font
-				(size 1.27 1.27)
-			)
-		)
-	)
-	(text "Was 20k"
-		(exclude_from_sim no)
-		(at 146.05 39.37 0)
-		(effects
-			(font
-				(size 1.27 1.27)
-			)
-		)
-	)
-	(text "Was 100k"
-		(exclude_from_sim no)
-		(at 171.45 16.51 0)
-		(effects
-			(font

Commit message: Exported BoM and Schematic
Other:
- company: (none) -> DMH Instruments
- title: (none) -> 5532 Output
- moved on the sheet: C23, C24, D33, D34, D43, D44, R84, R86, R87, R89, R92, R94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
