File: DMH_Output_PCB_Main/Output_Meter.kicad_sch (KiCad schematic)
At the start: 63 parts, among them Q1 BC558, Q2 BC558, U1 TL072, U2 LM339, U3 LM339, U4 LM339, U5 LM339, U6 LM339

Commit message: Adjusted output meter resistors
... and deleted unnecessary notes
Parts:
- removed R22, R25: 470R, Resistor_THT:R_Axial_DIN0207_L6.3mm_D2.5mm_P7.62mm_Horizontal, symbol Device:R_US
- R21, R23: value 75R -> 47R
Connections:
- net at D7.2 (A), U5.13: now also Q2.1 (C)
- net at D26.2 (A), U3.2: now also Q1.1 (C)
Changed lines of the file:
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@@
 	(wire
 		(pts
-			(xy 203.2 152.4) (xy 243.84 152.4)
+			(xy 203.2 152.4) (xy 254 152.4)
 		)
 		(stroke
@@
 	(wire
 		(pts
-			(xy 99.06 152.4) (xy 139.7 152.4)
-		)
-		(stroke
-			(width 0)
-			(type default)
-		)
-	)
-	(wire
-		(pts
 			(xy 179.07 60.96) (xy 182.88 60.96)
 		)
@@
 	(wire
 		(pts
-			(xy 88.9 152.4) (xy 91.44 152.4)
+			(xy 88.9 152.4) (xy 139.7 152.4)
 		)
 		(stroke
@@
 	(wire
 		(pts
-			(xy 254 152.4) (xy 251.46 152.4)
-		)
-		(stroke
-			(width 0)
-			(type default)
-		)
-	)
-	(wire
-		(pts
 			(xy 171.45 63.5) (xy 171.45 66.04)
 		)
@@
 	(symbol
 		(lib_id "Device:R_US")
-		(at 247.65 152.4 270)
-		(unit 1)
-		(body_style 1)
-		(exclude_from_sim no)
-		(in_bom yes)
-		(on_board no)
-		(in_pos_files yes)
-		(dnp no)
-		(property "Reference" "R25"
-			(at 247.65 158.75 90)
-			(show_name no)
-			(do_not_autoplace no)
-			(effects
-				(font
-					(size 1.27 1.27)
-				)
-			)
-		)
-		(property "Value" "470R"
-			(at 247.65 156.21 90)
-			(show_name no)
-			(do_not_autoplace no)
-			(effects
-				(font
-					(size 1.27 1.27)
-				)
-			)
-		)
-		(property "Footprint" "Resistor_THT:R_Axial_DIN0207_L6.3mm_D2.5mm_P7.62mm_Horizontal"
-			(at 247.396 153.416 90)
-			(hide yes)
-			(show_name no)
-			(do_not_autoplace no)
-			(effects
-				(font
-					(size 1.27 1.27)
-				)
-			)
-		)
-		(property "Datasheet" ""
-			(at 247.65 152.4 0)
-			(hide yes)
-			(show_name no)
-			(do_not_autoplace no)
-			(effects
-				(font
-					(size 1.27 1.27)
-				)
-			)
-		)
-		(property "Description" "Resistor, US symbol"
-			(at 247.65 152.4 0)
-			(hide yes)
-			(show_name no)
-			(do_not_autoplace no)
-			(effects
-				(font
-					(size 1.27 1.27)
-				)
-			)
-		)
-		(pin "2"
-		)
-		(pin "1"
-		)
-		(instances
-			(project "DMH_Output_PCB_Main"
-				(path "/58f4306d-5387-4983-bb08-41a2313fd315/91d96a83-7777-458d-a0c8-9961efcb16a5"
-					(reference "R25")
-					(unit 1)
-				)
-			)
-		)
-	)
-	(symbol
-		(lib_id "Device:R_US")
 		(at 171.45 135.89 180)
 		(unit 1)
@@
 			)
 		)
-		(property "Value" "75R"
+		(property "Value" "47R"
 			(at 251.46 128.2699 0)
 			(show_name no)
@@
 	)
 	(symbol
-		(lib_id "Device:R_US")
-		(at 95.25 152.4 90)
-		(mirror x)
-		(unit 1)
-		(body_style 1)
-		(exclude_from_sim no)
-		(in_bom yes)
-		(on_board no)
-		(in_pos_files yes)
-		(dnp no)
-		(property "Reference" "R22"
-			(at 95.25 158.75 90)
-			(show_name no)
-			(do_not_autoplace no)
-			(effects
-				(font
-					(size 1.27 1.27)
-				)
-			)
-		)
-		(property "Value" "470R"
-			(at 95.25 156.21 90)
-			(show_name no)
-			(do_not_autoplace no)
-			(effects
-				(font
-					(size 1.27 1.27)
-				)
-			)
-		)
-		(property "Footprint" "Resistor_THT:R_Axial_DIN0207_L6.3mm_D2.5mm_P7.62mm_Horizontal"
-			(at 95.504 153.416 90)
-			(hide yes)
-			(show_name no)
-			(do_not_autoplace no)
-			(effects
-				(font
-					(size 1.27 1.27)
-				)
-			)
-		)
-		(property "Datasheet" ""
-			(at 95.25 152.4 0)
-			(hide yes)
-			(show_name no)
-			(do_not_autoplace no)
-			(effects
-				(font
-					(size 1.27 1.27)
-				)
-			)
-		)
-		(property "Description" "Resistor, US symbol"
-			(at 95.25 152.4 0)
-			(hide yes)
-			(show_name no)
-			(do_not_autoplace no)
-			(effects
-				(font
-					(size 1.27 1.27)
-				)
-			)
-		)
-		(pin "2"
-		)
-		(pin "1"
-		)
-		(instances
-			(project "DMH_Output_PCB_Main"
-				(path "/58f4306d-5387-4983-bb08-41a2313fd315/91d96a83-7777-458d-a0c8-9961efcb16a5"
-					(reference "R22")
-					(unit 1)
-				)
-			)
-		)
-	)
-	(symbol
 		(lib_id "power:GND")
 		(at 88.9 50.8 0)
@@
 			)
 		)
-		(property "Value" "75R"
+		(property "Value" "47R"
 			(at 91.44 128.2699 0)
 			(show_name no)

Commit message: Exported BoM and Schematic
Other:
- company: (none) -> DMH Instruments
- title: (none) -> 5532 Output
Changed lines of the file:
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@@
 	(paper "A4")
 	(title_block
-		(comment 1 "PCB for 5 cm Kosmo format synthesizer module")
+		(title "5532 Output")
+		(date "2026-07-09")
+		(company "DMH Instruments")
+		(comment 1 "5 cm Kosmo format synthesizer module")
 	)
 	(text "Controls PCB"
