File: DMH_Output_PCB_Mezanine/Input_Meter.kicad_sch (KiCad schematic)
At the start: 29 parts, among them U20 TL072, U24 LM339, U25 LM339

Commit message: Adjusted output meter resistors
... and deleted unnecessary notes
Parts:
- R84: value 22K -> 22k
Other:
- note removed: "Was 100k"
- note removed: "Was 20k"
Changed lines of the file:
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@@
 		(comment 1 "PCB for 5 cm Kosmo format synthesizer module")
-	)
-	(circle
-		(center 171.45 22.86)
-		(radius 5.08)
-		(stroke
-			(width 0)
-			(type default)
-		)
-		(fill
-			(type none)
-		)
-	)
-	(circle
-		(center 57.15 22.86)
-		(radius 5.08)
-		(stroke
-			(width 0)
-			(type default)
-		)
-		(fill
-			(type none)
-		)
-	)
-	(circle
-		(center 146.05 45.72)
-		(radius 5.08)
-		(stroke
-			(width 0)
-			(type default)
-		)
-		(fill
-			(type none)
-		)
 	)
 	(rectangle
@@
 			(width 0.25)
 			(type dash)
-		)
-		(fill
-			(type none)
-		)
-	)
-	(circle
-		(center 31.75 45.72)
-		(radius 5.08)
-		(stroke
-			(width 0)
-			(type default)
 		)
 		(fill
@@
 		)
 	)
-	(text "Was 100k"
-		(exclude_from_sim no)
-		(at 57.15 16.51 0)
-		(effects
-			(font
-				(size 1.27 1.27)
-			)
-		)
-	)
-	(text "Was 20k"
-		(exclude_from_sim no)
-		(at 31.75 39.37 0)
-		(effects
-			(font
-				(size 1.27 1.27)
-			)
-		)
-	)
 	(text "3 = Green"
 		(exclude_from_sim no)
@@
 		(exclude_from_sim no)
 		(at 45.72 78.74 0)
-		(effects
-			(font
-				(size 1.27 1.27)
-			)
-		)
-	)
-	(text "Was 20k"
-		(exclude_from_sim no)
-		(at 146.05 39.37 0)
-		(effects
-			(font
-				(size 1.27 1.27)
-			)
-		)
-	)
-	(text "Was 100k"
-		(exclude_from_sim no)
-		(at 171.45 16.51 0)
 		(effects
 			(font
@@
 			)
 		)
-		(property "Value" "22K"
+		(property "Value" "22k"
 			(at 57.15 21.59 90)
 			(show_name no)
