File: DMH_Output_PCB_Mezanine/DMH_Output_PCB_Mezanine.kicad_sch (KiCad schematic)
At the start: 14 parts, among them J1 TRS_Jack_6.35mm_Sw, J2 TRS_Jack_6.35mm_Sw, J200 IDC_02x05, J21 Conn_01x02, J22 Conn_01x02, J24 Conn_01x02, J25 Conn_01x02, J3 TRS_Jack_6.35mm_Sw, J4 TRS_Jack_6.35mm_Sw, J5 TRS_Jack_6.35mm_Sw, J6 TRS_Jack_6.35mm_Sw, J7 TRS_Jack_6.35mm_Sw, J8 TRS_Jack_6.35mm_Sw, J9 TRS_Jack_6.35mm_Sw

Commit message: Added test points for easier calibration
Parts:
- added TP21, TP22, TP23, TP24: TestPoint, Connector_Pin:Pin_D1.0mm_L10.0mm, symbol Connector:TestPoint
Connections:
- net Balanced Line Driver/L_Bal_OUT_N_M: now also TP22.1
- net Balanced Line Driver/L_Bal_OUT_P_M: now also TP21.1
- net Balanced Line Driver/R_Bal_OUT_N_M: now also TP24.1
- net Balanced Line Driver/R_Bal_OUT_P_M: now also TP23.1
