File: DMH_Output_PCB_Controls/DMH_Output_PCB_Controls.kicad_pcb (KiCad board)
At the start: 2 copper layers, 48 x 121 mm, 89 parts, among them J10 Conn_01x06, J11 Conn_01x06_PinHeader, J12 Conn_01x06_PinHeader, J13 Conn_01x06, J21 Conn_01x02, J22 Conn_01x02, Q1 BC558, Q2 BC558, U2 LM339, U21 LM4040LP-10, U24 LM339, U25 LM339, U3 LM339, U4 LM339, U5 LM339, U6 LM339

Commit message: Adjusted output meter resistors
... and deleted unnecessary notes
Parts:
- removed R22, R25: 470R, Resistor_THT:R_Axial_DIN0207_L6.3mm_D2.5mm_P7.62mm_Horizontal
- R21, R23: value 75R -> 47R
Connections:
- Q1 pad 1: Net-(Q1-C) -> Net-(D26-A)
- Q2 pad 1: Net-(Q2-C) -> Net-(D7-A)
Routing:
- net Net-(D26-A): track 89.3 -> 116.5 mm
- net Net-(Q2-C): track 14.4 -> 0.00 mm
- net Net-(Q1-C): track 12.9 -> 0.00 mm
- net Net-(D7-A): track 99.0 -> 104.0 mm
Other:
- board text added: "Mk1.1 July 2026"
- board text removed: "Mk1.1 April 2026"
