File: DMH_Output_PCB_Controls/Balanced_line_driver.kicad_sch (KiCad schematic)
At the start: 38 parts, among them U10 NE5532, U9 NE5532

Commit message: Inverted line outputs hot and cold pins
... in order to avoid phase inversion at the TRS jack tip.
Connections:
- net L_Bal_OUT_N: now also C27.2, R101.2, R103.2; no longer C28.2, R100.2, R104.1
- net L_Bal_OUT_P: now also C28.2, R100.2, R104.1; no longer C27.2, R101.2, R103.2
- net R_Bal_OUT_N: now also C31.2, R115.2, R43.2; no longer C34.2, R106.2, R111.1
- net R_Bal_OUT_P: now also C34.2, R106.2, R111.1; no longer C31.2, R115.2, R43.2
Changed lines of the file:
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@@
 	(hierarchical_label "R_Bal_OUT_N"
+		(shape output)
+		(at 165.1 165.1 0)
+		(effects
+			(font
+				(size 1.27 1.27)
+			)
+			(justify left)
+		)
+	)
+	(hierarchical_label "R_Bal_OUT_P"
 		(shape output)
 		(at 165.1 215.9 0)
@@
 		)
 	)
-	(hierarchical_label "R_Bal_OUT_P"
-		(shape output)
-		(at 165.1 165.1 0)
-		(effects
-			(font
-				(size 1.27 1.27)
-			)
-			(justify left)
-		)
-	)
 	(hierarchical_label "L_Bal_OUT_P"
 		(shape output)
-		(at 165.1 50.8 0)
+		(at 165.1 101.6 0)
 		(effects
 			(font
@@
 	(hierarchical_label "L_Bal_OUT_N"
 		(shape output)
-		(at 165.1 101.6 0)
+		(at 165.1 50.8 0)
 		(effects
 			(font
